File: PCBS/Auxiliary-Charger/superbike-charger.sch (EAGLE design)
At the start: 20 parts, among them U1 BQ24125RHLR

Commit message: teensy board final draft
Parts:
- removed R_SYS: (no value), adafruit:R-US_R0805
- added V_OUT: LSP13, solpad:LSP13
- R_SNS: value .05R -> .05; device adafruit:R-US_R0805 -> rcl:R-US_R0402
Connections:
- net GND: no longer R_SYS.2
- net N$3: now also R_SNS.2, V_OUT.MP; no longer R_SNS.1, R_SYS.1
- net N$7: now also R_SNS.1; no longer R_SNS.2
Other:
- moved on the sheet: R_SNS
Changed lines of the file:
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@@
 <layers>
 <layer number="1" name="Top" color="4" fill="1" visible="no" active="no"/>
+<layer number="2" name="Route2" color="1" fill="3" visible="no" active="no"/>
+<layer number="3" name="Route3" color="4" fill="3" visible="no" active="no"/>
+<layer number="4" name="Route4" color="1" fill="4" visible="no" active="no"/>
+<layer number="5" name="Route5" color="4" fill="4" visible="no" active="no"/>
+<layer number="6" name="Route6" color="1" fill="8" visible="no" active="no"/>
+<layer number="7" name="Route7" color="4" fill="8" visible="no" active="no"/>
+<layer number="8" name="Route8" color="1" fill="2" visible="no" active="no"/>
+<layer number="9" name="Route9" color="4" fill="2" visible="no" active="no"/>
+<layer number="10" name="Route10" color="1" fill="7" visible="no" active="no"/>
+<layer number="11" name="Route11" color="4" fill="7" visible="no" active="no"/>
+<layer number="12" name="Route12" color="1" fill="5" visible="no" active="no"/>
+<layer number="13" name="Route13" color="4" fill="5" visible="no" active="no"/>
+<layer number="14" name="Route14" color="1" fill="6" visible="no" active="no"/>
+<layer number="15" name="Route15" color="4" fill="6" visible="no" active="no"/>
 <layer number="16" name="Bottom" color="1" fill="1" visible="no" active="no"/>
 <layer number="17" name="Pads" color="2" fill="1" visible="no" active="no"/>
@@
 <part name="GND2" library="supply1" library_urn="urn:adsk.eagle:library:371" deviceset="GND" device=""/>
 <part name="12.6V" library="battery" library_urn="urn:adsk.eagle:library:109" deviceset="SL340P" device="" package3d_urn="urn:adsk.eagle:package:4605/1"/>
-<part name="R_SNS" library="adafruit" library_urn="urn:adsk.eagle:library:420" deviceset="R-US_" device="R0805" package3d_urn="urn:adsk.eagle:package:6240566/1" value=".05R"/>
 <part name="R_ISET1" library="adafruit" library_urn="urn:adsk.eagle:library:420" deviceset="R-US_" device="R0805" package3d_urn="urn:adsk.eagle:package:6240566/1" value="10kR"/>
 <part name="R_ISET2" library="adafruit" library_urn="urn:adsk.eagle:library:420" deviceset="R-US_" device="R0805" package3d_urn="urn:adsk.eagle:package:6240566/1" value="10kR"/>
@@
 <part name="C5" library="adafruit" library_urn="urn:adsk.eagle:library:420" deviceset="C-US" device="C0805" package3d_urn="urn:adsk.eagle:package:6240337/1" value=".1uf"/>
 <part name="GND3" library="supply1" library_urn="urn:adsk.eagle:library:371" deviceset="GND" device=""/>
-<part name="R_SYS" library="adafruit" library_urn="urn:adsk.eagle:library:420" deviceset="R-US_" device="R0805" package3d_urn="urn:adsk.eagle:package:6240566/1"/>
-<part name="GND4" library="supply1" library_urn="urn:adsk.eagle:library:371" deviceset="GND" device=""/>
 <part name="LED1" library="adafruit" library_urn="urn:adsk.eagle:library:420" deviceset="LED" device="" package3d_urn="urn:adsk.eagle:package:6240563/1"/>
 <part name="LED2" library="adafruit" library_urn="urn:adsk.eagle:library:420" deviceset="LED" device="" package3d_urn="urn:adsk.eagle:package:6240563/1"/>
@@
 <part name="SUPPLY7" library="supply2" library_urn="urn:adsk.eagle:library:372" deviceset="GND" device=""/>
 <part name="GND5" library="supply1" library_urn="urn:adsk.eagle:library:371" deviceset="GND" device=""/>
+<part name="R_SNS" library="rcl" library_urn="urn:adsk.eagle:library:334" deviceset="R-US_" device="R0402" package3d_urn="urn:adsk.eagle:package:23547/3" value=".05"/>
+<part name="V_OUT" library="solpad" library_urn="urn:adsk.eagle:library:364" deviceset="LSP13" device="" package3d_urn="urn:adsk.eagle:package:26509/1"/>
 </parts>
 <sheets>
@@
 <attribute name="NAME" x="135.89" y="95.885" size="1.778" layer="95" rot="R180"/>
 </instance>
-<instance part="R_SNS" gate="G$1" x="139.7" y="96.52" smashed="yes" rot="R270">
-<attribute name="NAME" x="141.1986" y="100.33" size="1.778" layer="95" rot="R270"/>
-<attribute name="VALUE" x="136.398" y="100.33" size="1.778" layer="96" rot="R270"/>
-</instance>
 <instance part="R_ISET1" gate="G$1" x="53.34" y="71.12" smashed="yes">
 <attribute name="NAME" x="46.99" y="72.6186" size="1.778" layer="95"/>
@@
 <attribute name="VALUE" x="35.56" y="71.12" size="1.778" layer="96"/>
 </instance>
-<instance part="R_SYS" gate="G$1" x="149.86" y="101.6" smashed="yes">
-<attribute name="NAME" x="146.05" y="103.0986" size="1.778" layer="95"/>
-<attribute name="VALUE" x="146.05" y="98.298" size="1.778" layer="96"/>
-</instance>
-<instance part="GND4" gate="1" x="157.48" y="101.6" smashed="yes" rot="R90">
-<attribute name="VALUE" x="160.02" y="99.06" size="1.778" layer="96" rot="R90"/>
-</instance>
 <instance part="LED1" gate="G$1" x="50.8" y="104.14" smashed="yes">
 <attribute name="VALUE" x="56.515" y="99.568" size="1.778" layer="96" rot="R90"/>
@@
 <instance part="GND5" gate="1" x="129.54" y="88.9" smashed="yes">
 <attribute name="VALUE" x="127" y="86.36" size="1.778" layer="96"/>
+</instance>
+<instance part="R_SNS" gate="G$1" x="139.7" y="96.52" smashed="yes" rot="R90">
+<attribute name="NAME" x="138.2014" y="92.71" size="1.778" layer="95" rot="R90"/>
+<attribute name="VALUE" x="143.002" y="92.71" size="1.778" layer="96" rot="R90"/>
+</instance>
+<instance part="V_OUT" gate="1" x="147.32" y="101.6" smashed="yes" rot="R270">
+<attribute name="NAME" x="150.241" y="100.33" size="1.778" layer="95" rot="R270"/>
 </instance>
 </instances>
@@
 <wire x1="139.7" y1="109.22" x2="139.7" y2="101.6" width="0.1524" layer="91"/>
 <pinref part="C_OUT" gate="G$1" pin="1"/>
-<pinref part="R_SNS" gate="G$1" pin="1"/>
 <junction x="139.7" y="101.6"/>
 <wire x1="139.7" y1="101.6" x2="139.7" y2="104.14" width="0.1524" layer="91"/>
@@
 <pinref part="C2" gate="G$1" pin="1"/>
 <junction x="144.78" y="73.66"/>
-<pinref part="R_SYS" gate="G$1" pin="1"/>
+<pinref part="R_SNS" gate="G$1" pin="2"/>
+<pinref part="V_OUT" gate="1" pin="MP"/>
 <junction x="144.78" y="101.6"/>
 </segment>
@@
 <pinref part="C5" gate="G$1" pin="2"/>
 <pinref part="GND3" gate="1" pin="GND"/>
-</segment>
-<segment>
-<pinref part="R_SYS" gate="G$1" pin="2"/>
-<pinref part="GND4" gate="1" pin="GND"/>
 </segment>
 <segment>
@@
 <wire x1="119.38" y1="71.12" x2="139.7" y2="71.12" width="0.1524" layer="91"/>
 <pinref part="12.6V" gate="G$1" pin="+"/>
-<pinref part="R_SNS" gate="G$1" pin="2"/>
 <wire x1="139.7" y1="93.98" x2="139.7" y2="91.44" width="0.1524" layer="91"/>
 <junction x="139.7" y="91.44"/>
 <wire x1="139.7" y1="71.12" x2="139.7" y2="91.44" width="0.1524" layer="91"/>
-</segment>
-</net>
+<pinref part="R_SNS" gate="G$1" pin="1"/>
+</segment>
+</net>
